File: hw/ponictron.kicad_sch (KiCad schematic)
At the start: 53 parts, among them IC1 SHT40-BD1B-R2, IC2 MAX31328NELB+, IC3 PEC11S-929K-S0015, J1 FC68148S, J3 M20-7920642R, J4 SM04B-SRSS-TB_LF__SN__P_, J5 Conn_01x09, Q1 2SC5585TL, Q3 DMG2305UX-7, Q4 2SC5585TL, U1 RaspberryPi_Pico, U2 MCP4725A1T-E/CH, U3 LM358M, U4 TPS61040DBVR, U5 MPM3550EGLE

Commit message: Finish light control and power circuits
Parts:
- removed C1: 10uF, Capacitor_SMD:C_0603_1608Metric, symbol Device:C
- removed C2, C3: 22uF, Capacitor_SMD:C_0603_1608Metric, symbol Device:C
- removed L1: 10 uH, symbol Device:L
- removed R18: 875kΩ, Resistor_SMD:R_0603_1608Metric_Pad0.98x0.95mm_HandSolder, symbol Device:R
- removed U4: TPS61040DBVR, DBV0005A, symbol TPS61040:TPS61040DBVR
- added J2: RJCSE538001, RJCSE538001:AMPHENOL_RJCSE538001, symbol RJCSE538001:RJCSE538001
- added U4: DMP4015SSSQ-13, SO8_DIO, symbol DMP4015SSSQ-13:DMP4015SSSQ-13
- R16: value 100kΩ -> 1kΩ; LCSC Part # C103198 -> C15401
- R17: value 100kΩ -> 2kΩ; LCSC Part # C103198 -> C15401
Connections:
- net +12V: now also U3.8 (VCC), U4.1 (S), U4.2 (S), U4.3 (S); no longer J1.1, J1.2
- net +3.3V: no longer R16.2
- net GND: now also R16.2, J2.5, U4.4 (G); no longer R17.1
- net at U3.1 (OUT1): now also R17.1, J2.6
- net at U3.2 (IN1(-)): now also R16.1, R17.2
- new net: J1.1, J1.2, U4.5 (D), U4.6 (D), U4.7 (D), U4.8 (D)
Other:
- note added: "12V Power"
- note added: "Pico Power"
- note added: "Reverse voltage protection"
- note removed: "Power"
- moved on the sheet: C4, C5, J1, Q3, R19, U5

Commit message: Further progress on schematic
Parts:
- removed S1: RKB2SJK250SMTR_LFS, SamacSys_Parts:RKB2SJK250SMTRLFS, symbol SamacSys_Parts:RKB2SJK250SMTR_LFS
- added J6, J7, J8: B4B-PH-SM4-TB, B4B-PH-SM4-TB:JST_B4B-PH-SM4-TB, symbol B4B-PH-SM4-TB:B4B-PH-SM4-TB
- added R18, R20: 10kΩ, Resistor_SMD:R_0603_1608Metric_Pad0.98x0.95mm_HandSolder, symbol Device:R
- added R21: 4.7kΩ, Resistor_SMD:R_0603_1608Metric_Pad0.98x0.95mm_HandSolder, symbol Device:R
- added S1: TL3301BF260QJ, TL3301BF260QJ, symbol SamacSys_Parts:TL3301BF260QJ
Connections:
- net +12V: now also J6.2, J7.2
- net +3.3V: now also J4.2, J8.2, R18.2, R20.2, R21.1; no longer J4.3
- net GND: now also J4.1, J6.1, J7.1, J8.1, S1.4; no longer J4.4
- net SCL: now also J4.4, R10.2; no longer J4.1, R9.2
- net SDA: now also J4.3, R9.2; no longer J4.2, R10.2
- net FAN1: now reaches U1.21 (GPIO16)
- net FAN1: now also J6.4
- net FAN2: now reaches U1.22 (GPIO17)
- net FAN2: now also J7.4
- net MISO: now reaches U1.26 (GPIO20)
- net at U1.30 (RUN): now also S1.1
- net ANODE_L1_L2 renamed PROBE
- net PROBE: now also J8.3, R21.2
- net ANODE_L3 renamed TACH2
- net TACH2: now also J7.3, R20.1
- net EinkCS renamed DispCS
- net Enc_D: no longer names the net of IC3.D1 (COM), R11.1
- net IRQ renamed TACH1
- net TACH1: now also J6.3, R18.1
- new net: J8.SH1 (SHIELD), J8.SH2 (SHIELD__1)
- new net: J6.SH1 (SHIELD), J6.SH2 (SHIELD__1)
- new net: J7.SH1 (SHIELD), J7.SH2 (SHIELD__1)
Other:
- note added: "Fans"
- note added: "Probe"
- note added: "SPI Breakout"
- note added: "TODO: Add rocker switch for display"
- moved on the sheet: J2, J4, R10, R11, R15, R16, R17, R9, S2, U2, U3

Commit message: Add slider switch
Parts:
- added H5, H6, H7, H8: MountingHole_Pad, MountingHole:MountingHole_2.7mm_M2.5_DIN965_Pad, symbol Mechanical:MountingHole_Pad
- added J9: B4B-PH-SM4-TB, B4B-PH-SM4-TB:JST_B4B-PH-SM4-TB, symbol B4B-PH-SM4-TB:B4B-PH-SM4-TB
- added R22: 4.7kΩ, Resistor_SMD:R_0603_1608Metric_Pad0.98x0.95mm_HandSolder, symbol Device:R
- added S3: SLW-865144-2A-N-SMT-TR, SLW-865144-2A-N-SMT-TR:SW_SLW-865144-2A-N-SMT-TR, symbol SLW-865144-2A-N-SMT-TR:SLW-865144-2A-N-SMT-TR
Connections:
- net +3.3V: now also J9.2, R22.1
- net FAN1: now also U1.11 (GPIO8); no longer U1.21 (GPIO16)
- net FAN2: now also U1.12 (GPIO9); no longer U1.22 (GPIO17)
- net GND: now also H5.1, H6.1, H7.1, H8.1, J9.1, S3.1
- net MISO: now also J3.3
- net MOSI: now also J3.5
- net SCK: now also J3.7
- net TACH1: now also U1.14 (GPIO10); no longer U1.15 (GPIO11)
- net TACH2: now also U1.15 (GPIO11); no longer U1.16 (GPIO12)
- removed net GP14: J3.3, U1.14 (GPIO10)
- removed net GP8: J3.7, U1.11 (GPIO8)
- removed net GP9: J3.5, U1.12 (GPIO9)
- net PROBE renamed PROBE1
- net PROBE1: now also U1.16 (GPIO12); no longer U1.17 (GPIO13)
- new net: S3.2, U1.21 (GPIO16)
- new net: J9.SH1 (SHIELD), J9.SH2 (SHIELD__1)
- new net PROBE2: J9.3, R22.2, U1.17 (GPIO13)
Other:
- note added: "Adafruit 4694"
- note added: "Display activate"
- note added: "TODO: Switch to compat conn?"
- note removed: "TODO: Add rocker switch for display"
- moved on the sheet: J8, R21

Commit message: Further updates to schematic
Parts:
- removed J6, J7, J8, J9: B4B-PH-SM4-TB, B4B-PH-SM4-TB:JST_B4B-PH-SM4-TB, symbol B4B-PH-SM4-TB:B4B-PH-SM4-TB
- removed R22: 4.7kΩ, Resistor_SMD:R_0603_1608Metric_Pad0.98x0.95mm_HandSolder, symbol Device:R
- removed S1: TL3301BF260QJ, TL3301BF260QJ, symbol SamacSys_Parts:TL3301BF260QJ
- added C1, C2: 1uF, Capacitor_SMD:C_0603_1608Metric, symbol Device:C
- added J2: MSD-11-A, MSD-11-A:CUI_MSD-11-A, symbol MSD-11-A:MSD-11-A
- added J3, J6: 470531000, CONN_SD-47053-001_H10p00_MOL, symbol 0470531000:470531000
- added J4, J5, J7: B3B-PH-SM4-TB_LF__SN_, B3B-PH-SM4-TB_LF__SN_:JST_B3B-PH-SM4-TB_LF__SN_, symbol B3B-PH-SM4-TB_LF__SN_:B3B-PH-SM4-TB_LF__SN_
- added R3, R4, R5, R6, R7, R8: 47kΩ, Resistor_SMD:R_0603_1608Metric_Pad0.98x0.95mm_HandSolder, symbol Device:R
- added TP2: RTC_INT, TestPoint:TestPoint_Pad_1.5x1.5mm, symbol Connector:TestPoint
- IC3: footprint PEC11S929KS0015 -> SamacSys_Parts:PEC11S929KS0015
- J11: renamed from J1; footprint FC68148S_CLF -> FC68148S:FC68148S_CLF
- R24: renamed from R2; footprint TRANS_2SA2018_ROM -> 2SA2018TL:TRANS_2SA2018_ROM
- R25: renamed from R12; footprint TRANS_2SA2018_ROM -> 2SA2018TL:TRANS_2SA2018_ROM
- S1: renamed from S9; footprint TL3301BF260QJ -> SamacSys_Parts:TL3301BF260QJ
- S2: footprint TL3301BF260QJ -> SamacSys_Parts:TL3301BF260QJ
- TP1: renamed from TP2; value TestPoint -> Bootsel
- U1: renamed from U3; footprint 8-SOP_OSI -> LM358M:8-SOP_OSI
- U2: footprint SOT-23-6_MC_MCH -> MCP4725A1T_E_CH:SOT-23-6_MC_MCH
- U4: footprint SO8_DIO -> DMP4015SSSQ-13:SO8_DIO
- renumbered C13 to C3, C14 to C4, C15 to C5, C16 to C6, C5 to C7, C4 to C8, J2 to J1, J5 to J10, J3 to J8, J4 to J9, LS2 to LS1, Q4 to Q1, Q3 to Q2, Q1 to Q3, R17 to R1, R18 to R10, R21 to R11, R20 to R12, R3 to R13, R4 to R14, R5 to R15, R7 to R16, R8 to R17, R9 to R18, R10 to R19, R16 to R2, R11 to R20, R1 to R21, R6 to R22, R19 to R23, R13 to R26, R14 to R27, R15 to R9, U1 to U3
Connections:
- net PROBE2 is gone; now on net TACH2: U3.17 (GPIO13)
- net +12V: now also J3.2, J6.2
- net +3.3V: now also C1.2, C2.2, J2.P4 (VDD), J4.2, J5.2, J7.2, R3.1, R4.2, R5.1, R6.2, R7.1, R8.2
- net ADC0: now also J5.1; no longer J8.4
- net Buzzer: now also U3.29 (GPIO22); no longer U3.4 (GPIO2)
- net Enc_E: now also U3.4 (GPIO2); no longer U3.29 (GPIO22)
- net GND: now also C1.1, C2.1, J2.G1 (COVER_GND), J2.G2 (COVER_GND__1), J2.P6 (VSS), J3.1, J4.1, J5.3, J6.1, J7.1
- net MISO: now also J2.P7 (DAT0), R4.1
- net MOSI: now also J2.P3 (CMD), R6.1
- net SCK: now also J2.P5 (CLK), R8.1
- net TACH1: now also U3.16 (GPIO12), J3.3; no longer U3.14 (GPIO10)
- net TACH2: now also J6.3; no longer U3.15 (GPIO11)
- net msdCS: now reaches U3.22 (GPIO17)
- net msdCS: now also J2.P2 (CD/DAT3), R7.2
- net FAN1 renamed msdDet
- net msdDet: now also J2.CD, J2.WP
- net FAN2 renamed msdDAT1
- net msdDAT1: now also J2.P8 (DAT1), R3.2
- net PROBE1 renamed onewire
- net onewire: now also U3.5 (GPIO3), J4.3, J7.3; no longer U3.16 (GPIO12)
- net RTC_INT: no longer names the net of IC2.3 (~{INT}/SQW), R15.2
- net RTC_INT: now also TP2.1; no longer U3.5 (GPIO3)
- new net FAN: J3.4, J6.4, U3.15 (GPIO11)
- new net msdDAT2: J2.P1 (DAT2), R5.2, U3.14 (GPIO10)
Other:
- note added: "MicroSD"
- note added: "TDS Sensor"
- note removed: "Reset"
- note removed: "SPI Breakout"
- note removed: "TODO: Switch to compat conn?"
- moved on the sheet: C3, C4, C5, C6, C7, C8, H1, H2, H3, H4, H5, H6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

Commit message: Add expander
Parts:
- removed H5, H6, H7, H8: MountingHole_Pad, MountingHole:MountingHole_2.7mm_M2.5_DIN965_Pad, symbol Mechanical:MountingHole_Pad
- removed J10: Conn_01x09, Connector_PinHeader_2.54mm:PinHeader_1x09_P2.54mm_Vertical, symbol Connector_Generic:Conn_01x09
- removed S3: SLW-865144-2A-N-SMT-TR, SLW-865144-2A-N-SMT-TR:SW_SLW-865144-2A-N-SMT-TR, symbol SLW-865144-2A-N-SMT-TR:SLW-865144-2A-N-SMT-TR
- added C10: 0.1uF, Capacitor_SMD:C_0603_1608Metric, symbol Device:C
- added C11, C9: 1uF, Capacitor_SMD:C_0603_1608Metric, symbol Device:C
- added H10, H11, H12, H9: MountingHole_Pad, MountingHole:MountingHole_2.7mm_M2.5_DIN965_Pad, symbol Mechanical:MountingHole_Pad
- added J12: Conn_01x10, symbol Connector_Generic:Conn_01x10
- added R28, R29, R30, R31, R32, R33: 10kΩ, Resistor_SMD:R_0603_1608Metric_Pad0.98x0.95mm_HandSolder, symbol Device:R
- added U6: MCP23017_SO, Package_SO:SOIC-28W_7.5x17.9mm_P1.27mm, symbol Interface_Expansion:MCP23017_SO
- C1: value 1uF -> 0.1uF
Connections:
- net +3.3V: now also C10.2, C11.2, C9.2, J12.2 (Pin_2), R28.2, R29.2, R30.2, U6.9 (VDD)
- net DispCS: now also U3.22 (GPIO17), J12.6 (Pin_6)
- net Enc_E: now also U6.3 (GPB2)
- net FAN: now also U3.16 (GPIO12); no longer U3.15 (GPIO11)
- net GND: now also C10.1, C11.1, C9.1, H10.1, H11.1, H12.1, H9.1, J12.1 (Pin_1), R31.1, R32.1, R33.1, U6.10 (VSS)
- net MOSI: now also J12.7 (Pin_7)
- net SCK: now also J12.9 (Pin_9)
- net SCL: now also U6.12 (SCK)
- net SDA: now also U6.13 (SDA)
- net TACH1: no longer U3.16 (GPIO12)
- net TACH2: no longer U3.17 (GPIO13)
- net msdCS: now also U3.14 (GPIO10); no longer U3.22 (GPIO17)
- net msdDAT1: now also U3.11 (GPIO8); no longer U3.12 (GPIO9)
- net msdDAT2: now also U3.12 (GPIO9); no longer U3.14 (GPIO10)
- net msdDet: now also U3.15 (GPIO11), U6.4 (GPB3); no longer U3.11 (GPIO8)
- net at S1.1: now also U6.2 (GPB1); no longer U3.19 (GPIO14)
- net at S2.1: now also U6.1 (GPB0); no longer U3.20 (GPIO15)
- net DispRST: now reaches U3.21 (GPIO16)
- net DispRST: now also J12.4 (Pin_4), U6.21 (GPA0)
- net GP6: no longer names the net of J8.11
- net GP6: no longer U3.9 (GPIO6)
- net GP7: no longer names the net of J8.9
- net GP7: no longer U3.10 (GPIO7)
- new net: R33.2, U6.15 (A0)
- new net: R32.2, U6.16 (A1)
- new net: R31.2, U6.17 (A2)
- new net: R30.1, U6.18 (~{RESET})
- new net INTA: R28.1, U3.9 (GPIO6), U6.19 (INTB)
- new net INTB: R29.1, U3.10 (GPIO7), U6.20 (INTA)
Other:
- note added: "Adafruit 1480"
- note added: "Expander"
- note removed: "Display activate"
- moved on the sheet: C1, C2, C3, C4, C5, C6, C7, C8, H1, H2, H3, H4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

Commit message: Remove expander, switch to TFT display, ready for board layout
Parts:
- removed C7: 4.7uF, Capacitor_SMD:C_0603_1608Metric, symbol Device:C
- removed J6: 470531000, CONN_SD-47053-001_H10p00_MOL, symbol 0470531000:470531000
- removed R10, R12, R28, R29, R30, R31, R32, R33: 10kΩ, Resistor_SMD:R_0603_1608Metric_Pad0.98x0.95mm_HandSolder, symbol Device:R
- removed U6: MCP23017_SO, Package_SO:SOIC-28W_7.5x17.9mm_P1.27mm, symbol Interface_Expansion:MCP23017_SO
- added C11, C12, C15, C18: 10uF, Capacitor_SMD:C_0603_1608Metric, symbol Device:C
- added C13, C14: 0.1uF, Capacitor_SMD:C_0603_1608Metric, symbol Device:C
- added C16: 22uF, Capacitor_SMD:C_0603_1608Metric, symbol Device:C
- added J8: 470531000, CONN_SD-47053-001_H10p00_MOL, symbol 0470531000:470531000
- added S3: TL3301BF260QJ, SamacSys_Parts:TL3301BF260QJ, symbol SamacSys_Parts:TL3301BF260QJ
- C1: renamed from C11; value 1uF -> 10uF
- C3: renamed from C2; value 1uF -> 10uF
- C4: renamed from C3; value 1uF -> 0.1uF
- C5: renamed from C4; value 1uF -> 0.1uF
- C6: renamed from C5; value 1uF -> 0.1uF
- C7: renamed from C6; value 1uF -> 0.1uF
- C8: value 1uF -> 10uF
- C9: value 1uF -> 0.1uF
- renumbered C1 to C2, H9 to H1, H10 to H2, H11 to H3, H12 to H4, H1 to H5, H2 to H6, H3 to H7, H4 to H8, J9 to J10, J12 to J2, J2 to J3, J3 to J5, J5 to J6, J8 to J9, R11 to R10, R13 to R11, R14 to R12, R15 to R13, R16 to R14, R17 to R15, R18 to R16, R19 to R17, R20 to R18, R21 to R19, R22 to R20, R23 to R21, R24 to R22, R25 to R23, R26 to R24, R27 to R25, R9 to R6, R6 to R7, R7 to R8, R8 to R9, S2 to S1, S1 to S2, U3 to U1, U1 to U2, U2 to U3, U5 to U4, U4 to U5
Connections:
- net INTA is gone; now on net GP6: U1.9 (GPIO6)
- net INTB is gone; now on net GP7: U1.10 (GPIO7)
- net +12V: now also C9.2, C12.2, C13.2, C18.2, J8.2
- net +3.3V: now also C8.1, C11.1, C14.2, C15.2; no longer C9.2
- net FAN: now also J8.4
- net GND: now also C11.2, C12.1, C13.1, C14.1, C15.1, C16.1, C18.1, J8.1, S3.4
- net BUT1: now reaches S1.1
- net BUT1: now also U1.17 (GPIO13)
- net BUT2: now reaches S2.1
- net BUT2: now also U1.19 (GPIO14)
- net at Q2.3 (D), U4.5 (VOUT): now also C16.2; no longer C8.1
- net BUT3: now reaches U1.20 (GPIO15)
- net BUT3: now also S3.1
- net GP6: now reaches J9.11
- net GP7: now reaches J9.9
- net TACH1: no longer names the net of J5.3
Other:
- note added: "Buttons"
- note added: "Probes"
- note removed: "Adafruit 4694"
- note removed: "Expander"
- note removed: "Probe"
- moved on the sheet: C4, H1, H2, H3, H4, IC2, J2, J3, J4, J5, R10, R13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

Commit message: Starting board layout
Parts:
- removed J9: M20-7920642R, SamacSys_Parts:M207920642R, symbol SamacSys_Parts:M20-7920642R
- removed S3: TL3301BF260QJ, SamacSys_Parts:TL3301BF260QJ, symbol SamacSys_Parts:TL3301BF260QJ
- added J6: Conn_01x10, Connector_PinHeader_2.54mm:PinHeader_1x10_P2.54mm_Vertical, symbol Connector_Generic:Conn_01x10
- added J7, J8: B3B-PH-SM4-TB_LF__SN_, B3B-PH-SM4-TB_LF__SN_:JST_B3B-PH-SM4-TB_LF__SN_, symbol B3B-PH-SM4-TB_LF__SN_:B3B-PH-SM4-TB_LF__SN_
- added TP2: ADC_VREF, TestPoint:TestPoint_Pad_1.5x1.5mm, symbol Connector:TestPoint
- J2: footprint (none) -> Connector_PinHeader_2.54mm:PinHeader_1x10_P2.54mm_Vertical
- J3: footprint MSD-11-A:CUI_MSD-11-A -> MSD_11_A:CUI_MSD-11-A
- LS1: footprint CPT-1203-03-SMT-TR:XDCR_CPT-1203-03-SMT-TR -> CPT_1203_03_SMT_TR:XDCR_CPT-1203-03-SMT-TR
- renumbered C4 to C10, C7 to C11, C8 to C12, C18 to C13, C9 to C14, C16 to C15, C14 to C16, C15 to C17, C13 to C3, C12 to C4, C3 to C5, C10 to C6, C5 to C7, C6 to C8, C11 to C9, J7 to J10, J8 to J11, J10 to J12, J11 to J13, J6 to J9, R10 to R1, R9 to R10, R1 to R2, R2 to R3, R3 to R4, R4 to R5, R5 to R6, R6 to R7, R7 to R8, R8 to R9, TP2 to TP3
Connections:
- net +3.3V: now also J6.10 (Pin_10), J7.2, J8.2
- net ADC1: now also J8.1
- net ADC2: now also J7.1
- net GND: now also J6.1 (Pin_1); no longer J9.3
- net GP6: now also J6.6 (Pin_6)
- net GP7: now also J6.5 (Pin_5)
- net MISO: now also J6.2 (Pin_2)
- net MOSI: now also J6.3 (Pin_3)
- net SCK: now also J6.4 (Pin_4)
- net SCL: now also J6.8 (Pin_8)
- net SDA: now also J6.9 (Pin_9)
- net ADC_VREF: no longer names the net of U1.35 (ADC_VREF)
- net ADC_VREF: now also TP2.1
- net AGND renamed GNDA
- net GNDA: now also J9.3, J7.3, J8.3
- net BUT3 renamed GP15
- net GP15: now also J6.7 (Pin_7)
Other:
- note added: "Analog Sensors"
- note removed: "TDS Sensor"
- moved on the sheet: J9, S1, S2

Commit message: Create board layout
Parts:
- J2, J6: footprint Connector_PinHeader_2.54mm:PinHeader_1x10_P2.54mm_Vertical -> Connector_PinSocket_2.54mm:PinSocket_1x10_P2.54mm_Vertical
- Q2: renamed from R22; footprint 2SA2018TL:TRANS_2SA2018_ROM -> TRANS_2SA2018_ROM
- Q4: renamed from R23; footprint 2SA2018TL:TRANS_2SA2018_ROM -> TRANS_2SA2018_ROM
- U4: footprint Package_LGA:MPS_LGA-18-10EP_12x12mm_P3.3mm -> MPM3550EGLE:MPM3550EGLE
- renumbered Q2 to Q3, Q3 to Q5, R24 to R22, R25 to R23
Connections:
- net +3.3V: now also J6.9 (Pin_9)
- net BUT1: now also U1.15 (GPIO11); no longer U1.17 (GPIO13)
- net BUT2: now also U1.14 (GPIO10); no longer U1.19 (GPIO14)
- net Buzzer: now also U1.27 (GPIO21); no longer U1.29 (GPIO22)
- net DispCS: no longer U1.27 (GPIO21)
- net DispRST: now also U1.17 (GPIO13); no longer U1.21 (GPIO16)
- net FAN: now also U1.29 (GPIO22); no longer U1.16 (GPIO12)
- net GND: now also J6.2 (Pin_2), J6.3 (Pin_3)
- net GP6: now also J6.8 (Pin_8); no longer J6.6 (Pin_6)
- net GP7: now also J6.7 (Pin_7); no longer J6.5 (Pin_5)
- net MISO: now also J6.5 (Pin_5), U1.21 (GPIO16); no longer J6.2 (Pin_2), U1.26 (GPIO20)
- net MOSI: now also J6.4 (Pin_4); no longer J6.3 (Pin_3)
- net SCK: now also J6.6 (Pin_6); no longer J6.4 (Pin_4)
- net SCL: no longer J6.8 (Pin_8)
- net SDA: no longer J6.9 (Pin_9)
- net msdCS: now also U1.26 (GPIO20); no longer U1.14 (GPIO10)
- net msdDAT1: now also U1.20 (GPIO15); no longer U1.11 (GPIO8)
- net msdDAT2: now also U1.19 (GPIO14); no longer U1.12 (GPIO9)
- net msdDet: now also U1.16 (GPIO12); no longer U1.15 (GPIO11)
- net BlitePWM: now reaches J2.10 (Pin_10)
- net BlitePWM: now also U1.12 (GPIO9)
- net DispD/C: now reaches J2.3 (Pin_3)
- net DispD/C: now also U1.11 (GPIO8)
- removed net GP15: J6.7 (Pin_7), U1.20 (GPIO15)
