File: hw/ponictron.kicad_sch (KiCad schematic)
At the start: 75 parts, among them IC1 SHT40-BD1B-R2, IC2 MAX31328NELB+, IC3 PEC11S-929K-S0015, J1 RJCSE538001, J10 B3B-PH-SM4-TB_LF__SN_, J11 470531000, J12 SM04B-SRSS-TB_LF__SN__P_, J13 FC68148S, J2 Conn_01x10, J3 MSD-11-A, J4 B3B-PH-SM4-TB_LF__SN_, J5 470531000, J6 Conn_01x10, J7 B3B-PH-SM4-TB_LF__SN_, J8 B3B-PH-SM4-TB_LF__SN_, J9 B3B-PH-SM4-TB_LF__SN_, Q1 DMG2305UX-7, U1 RaspberryPi_Pico, U2 LM358M, U3 MCP4725A1T-E/CH, U4 AP63203WU-7, U5 NC7WZ14P6X, U6 DMP4015SSSQ-13

Commit message: Various fixes for schematic issues
Parts:
- removed H1, H2, H3, H4: MountingHole_Pad, 78614015360:WE-SMSA_78614015360, symbol 78614015360:WE-SMSA_M3
- removed IC3: PEC11S-929K-S0015, SamacSys_Parts:PEC11S929KS0015, symbol SamacSys_Parts:PEC11S-929K-S0015
- removed R10: 47kΩ, Resistor_SMD:R_0603_1608Metric_Pad0.98x0.95mm_HandSolder, symbol Device:R
- removed R11, R12, R14, R15: 10kΩ, Resistor_SMD:R_0603_1608Metric_Pad0.98x0.95mm_HandSolder, symbol Device:R
- removed R18: 1kΩ, Resistor_SMD:R_0603_1608Metric_Pad0.98x0.95mm_HandSolder, symbol Device:R
- removed S1, S2: TL3301BF260QJ, SamacSys_Parts:TL3301BF260QJ, symbol SamacSys_Parts:TL3301BF260QJ
- removed U2: LM358M, LM358M:8-SOP_OSI, symbol LM358M:LM358M
- added MP1, MP2, MP3, MP4: WA-SMSI_9774XXX151, WA-SMSI_9774100151:WA-SMSI_9774100151, symbol WA-SMSI_9774XXX151:WA-SMSI_9774XXX151
- added Q2: BSS138, Package_TO_SOT_SMD:SOT-23, symbol Transistor_FET:BSS138
- added R20: 1kΩ, Resistor_SMD:R_0603_1608Metric_Pad0.98x0.95mm_HandSolder, symbol Device:R
- added S1, S3: PTS647SM70SMTR2LFS, PTS647SM38SMTR2LFS, symbol SamacSys_Parts:PTS647SM70SMTR2LFS
- added U7: MCP6001-OT, Package_TO_SOT_SMD:SOT-23-5, symbol Amplifier_Operational:MCP6001-OT
- C7: value 0.1uF -> 10uF
- R2: value 2kΩ -> 83Ω
- R3: value 1kΩ -> 32kΩ
- R4, R5, R6, R8, R9: value 47kΩ -> 10kΩ
Connections:
- net +12V: no longer C3.2, C4.2
- net +3.3V: now also C3.2, C4.2, C7.1, C8.1, U7.5 (V+)
- net BUT1: now also S3.3
- net BUT2: now also S1.3
- net GND: now also C7.2, C8.2, J13.1, J13.2, R2.2, MP1.1, MP2.1, MP3.1, MP4.1, R20.2, S1.2, S3.2, U7.2 (V-); no longer C7.1, C8.1, J13.4, R3.2
- net at J1.6: now also Q2.3 (D); no longer R2.1
- net at R3.1: now also U3.1 (VOUT); no longer R2.2
- net at U6.5 (D), U6.6 (D), U6.7 (D)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: now also J13.4; no longer J13.1, J13.2
- net Enc_A1: no longer names the net of U1.2 (GPIO1)
- net Enc_B1 renamed FAN2
- net FAN2: now also J11.4
- net Enc_E: no longer names the net of U1.4 (GPIO2)
- net FAN renamed FAN1
- net FAN1: no longer J11.4
- net msdDAT1: no longer names the net of J3.P8 (DAT1), R4.2
- net msdDAT1: no longer U1.20 (GPIO15)
- net msdDAT2: no longer names the net of J3.P1 (DAT2), R6.2
- net msdDAT2: no longer U1.19 (GPIO14)
- new net: Q2.1 (G), U7.1
- new net: Q2.2 (S), R2.1, U7.4 (-)
- new net: R20.1, R3.2, U7.3 (+)
Other:
- note added: "1.2 mA is max current draw of LED sink 0 V -> MOSFET closed -> 0 A -> max brightness 0.1 V / 1.2 mA = 83 Ω 0.1 V -> max current draw -> minimum brightness"
- note added: "The 83 Ω resistor is what causes the MOSFET to target 0.1 V, given the 1.2 mA. Which in turn drives the 1.2 mA current, Which in turn causes the 10 V drop at the LED driver. You want to target as low of a voltage as possible (0.1 V) so that the required sensing resistance is as low as possible because the 83 Ω gets added to the 8300 Ω 10 V / 8383 Ω = 1.19 mA, so you get as close as possible to ma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"
- note added: "There must be a roughly 8.3 kΩ resistor on the LED driver side So at 0 mA current draw, there is zero voltage drop, so the LED driver stays at 10 V. At 1.2 mA, 1.2/1000 * 8300 = 10 V, so there is a 10 V drop."
- note added: "linear op-amp sink"
- note added: "voltage divider, 3.3V -> 0.1V"
- note removed: "Encoder"
- moved on the sheet: C1, C10, C11, C12, C2, C3, C4, C9, IC1, IC2, J1, J13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

Commit message: Finish schematic and board layout changes
Parts:
- removed U5: NC7WZ14P6X, SC70-6_ONS, symbol NC7WZ14P6X:NC7WZ14P6X
- added TP1: GP10, TestPoint:TestPoint_Pad_1.5x1.5mm, symbol Connector:TestPoint
- added U6: SN74LVC2G240DCUR, SN74LVC2G240DCUR:SN74LVC2G240DCUR, symbol SN74LVC2G240DCUR:SN74LVC2G240DCUR
- renumbered C2 to C1, C1 to C2, C4 to C3, C3 to C4, C7 to C5, C8 to C6, C5 to C7, C6 to C8, H5 to H1, H6 to H2, H7 to H3, H8 to H4, Q2 to Q1, Q1 to Q2, R9 to R10, R13 to R11, R16 to R12, R17 to R13, R19 to R14, R7 to R2, R20 to R4, R4 to R5, R2 to R6, R5 to R7, R6 to R8, R8 to R9, S3 to S1, S1 to S2, TP1 to TP2, TP2 to TP3, TP3 to TP4, U3 to U2, U7 to U3, U6 to U5
Connections:
- net +3.3V: now also U6.8 (VCC); no longer J6.9 (Pin_9)
- net BUT1: now also U1.4 (GPIO2); no longer U1.15 (GPIO11)
- net BUT2: now also U1.2 (GPIO1); no longer U1.14 (GPIO10)
- net Buzzer: now also U1.1 (GPIO0), U6.2 (1A); no longer U1.27 (GPIO21)
- net FAN2: now also U1.27 (GPIO21); no longer U1.1 (GPIO0)
- net GND: now also U6.4 (GND); no longer J6.2 (Pin_2), J6.3 (Pin_3)
- net GP6: now also J6.9 (Pin_9); no longer J6.8 (Pin_8)
- net GP7: now also J6.8 (Pin_8); no longer J6.7 (Pin_7)
- net GP14: now reaches U1.19 (GPIO14)
- net GP14: now also J6.3 (Pin_3)
- net GP15: now reaches U1.20 (GPIO15)
- net GP15: now also J6.2 (Pin_2)
- net at LS1.P: now also U6.3 (2Y)
- net at R14.1: now also U6.5 (2A), U6.6 (1Y)
- new net: TP1.1, U1.14 (GPIO10)
- new net GP11: J6.7 (Pin_7), U1.15 (GPIO11)
Other:
- moved on the sheet: C15, C17, LS1, R1, R14

Commit message: Update schematic and board layout
Parts:
- removed TP1: GP10, TestPoint:TestPoint_Pad_1.5x1.5mm, symbol Connector:TestPoint
Connections:
- net BUT1: now also U1.5 (GPIO3); no longer U1.4 (GPIO2)
- net BUT2: now also U1.4 (GPIO2); no longer U1.2 (GPIO1)
- net onewire: now also U1.14 (GPIO10); no longer U1.5 (GPIO3)
- net Buzzer_EN: now reaches U6.1 (1OEN)
- net Buzzer_EN: now also U1.2 (GPIO1), U6.7 (2OEN)
Changed lines of the file:
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@@
 	(wire
 		(pts
-			(xy 43.18 129.54) (xy 52.07 129.54)
-		)
-		(stroke
-			(width 0)
-			(type default)
-		)
-	)
-	(wire
-		(pts
 			(xy 173.99 177.8) (xy 200.66 177.8)
 		)
@@
 	(wire
 		(pts
-			(xy 483.87 311.15) (xy 501.65 311.15)
-		)
-		(stroke
-			(width 0)
-			(type default)
-		)
-	)
-	(wire
-		(pts
 			(xy 80.01 83.82) (xy 80.01 86.36)
 		)
@@
 	(wire
 		(pts
+			(xy 496.57 323.85) (xy 496.57 313.69)
+		)
+		(stroke
+			(width 0)
+			(type default)
+		)
+	)
+	(wire
+		(pts
 			(xy 394.97 280.67) (xy 421.64 280.67)
 		)
@@
 	(wire
 		(pts
+			(xy 496.57 313.69) (xy 501.65 313.69)
+		)
+		(stroke
+			(width 0)
+			(type default)
+		)
+	)
+	(wire
+		(pts
 			(xy 389.89 82.55) (xy 393.7 82.55)
 		)
@@
 	(wire
 		(pts
+			(xy 501.65 323.85) (xy 496.57 323.85)
+		)
+		(stroke
+			(width 0)
+			(type default)
+		)
+	)
+	(wire
+		(pts
 			(xy 403.86 194.31) (xy 403.86 190.5)
 		)
@@
 	(wire
 		(pts
+			(xy 29.21 111.76) (xy 29.21 129.54)
+		)
+		(stroke
+			(width 0)
+			(type default)
+		)
+	)
+	(wire
+		(pts
 			(xy 519.43 120.65) (xy 521.97 120.65)
 		)
@@
 	(wire
 		(pts
-			(xy 29.21 111.76) (xy 52.07 111.76)
-		)
-		(stroke
-			(width 0)
-			(type default)
-		)
-	)
-	(wire
-		(pts
 			(xy 403.86 210.82) (xy 403.86 207.01)
 		)
@@
 	(wire
 		(pts
+			(xy 492.76 311.15) (xy 501.65 311.15)
+		)
+		(stroke
+			(width 0)
+			(type default)
+		)
+	)
+	(wire
+		(pts
 			(xy 59.69 299.72) (xy 60.96 299.72)
 		)
@@
 	(wire
 		(pts
+			(xy 29.21 129.54) (xy 52.07 129.54)
+		)
+		(stroke
+			(width 0)
+			(type default)
+		)
+	)
+	(wire
+		(pts
 			(xy 429.26 80.01) (xy 434.34 80.01)
 		)
@@
 		)
 	)
+	(label "Buzzer_EN"
+		(at 52.07 106.68 180)
+		(effects
+			(font
+				(size 1.27 1.27)
+			)
+			(justify right bottom)
+		)
+	)
 	(label "SDA"
 		(at 394.97 278.13 0)
@@
 	)
 	(label "BUT2"
-		(at 52.07 106.68 180)
+		(at 52.07 109.22 180)
 		(effects
 			(font
@@
 	)
 	(label "onewire"
-		(at 44.45 111.76 0)
+		(at 52.07 129.54 180)
 		(effects
 			(font
 				(size 1.27 1.27)
 			)
-			(justify left bottom)
+			(justify right bottom)
 		)
 	)
@@
 		)
 	)
+	(label "Buzzer_EN"
+		(at 496.57 313.69 180)
+		(effects
+			(font
+				(size 1.27 1.27)
+			)
+			(justify right bottom)
+		)
+	)
 	(label "DispCS"
 		(at 189.23 88.9 0)
@@
 	)
 	(label "Buzzer"
-		(at 483.87 311.15 0)
+		(at 492.76 311.15 180)
 		(effects
 			(font
 				(size 1.27 1.27)
 			)
-			(justify left bottom)
+			(justify right bottom)
 		)
 	)
@@
 	)
 	(label "BUT1"
-		(at 52.07 109.22 180)
+		(at 52.07 111.76 180)
 		(effects
 			(font
@@
 					(unit 1)
 				)
-			)
-		)
-	)
-	(symbol
-		(lib_id "Connector:TestPoint")
-		(at 43.18 129.54 90)
-		(unit 1)
-		(exclude_from_sim no)
-		(in_bom no)
-		(on_board yes)
-		(dnp no)
-		(fields_autoplaced yes)
-		(property "Reference" "TP1"
-			(at 39.878 124.46 90)
-			(effects
-				(font
-					(size 1.27 1.27)
-				)
-			)
-		)
-		(property "Value" "GP10"
-			(at 39.878 127 90)
-			(effects
-				(font
-					(size 1.27 1.27)
-				)
-			)
-		)
-		(property "Footprint" "TestPoint:TestPoint_Pad_1.5x1.5mm"
-			(at 43.18 124.46 0)
-			(effects
-				(font
-					(size 1.27 1.27)
-				)
-				(hide yes)
-			)
-		)
-		(property "Datasheet" "~"
-			(at 43.18 124.46 0)
-			(effects
-				(font
-					(size 1.27 1.27)
-				)
-				(hide yes)
-			)
-		)
-		(property "Description" "test point"
-			(at 43.18 129.54 0)
-			(effects
-				(font
-					(size 1.27 1.27)
-				)
-				(hide yes)
-			)
-		)
-		(property "Availability" ""
-			(at 43.18 129.54 0)
-			(effects
-				(font
-					(size 1.27 1.27)
-				)
-				(hide yes)
-			)
-		)
-		(property "Check_prices" ""
-			(at 43.18 129.54 0)
-			(effects
-				(font
-					(size 1.27 1.27)
-				)
-				(hide yes)
-			)
-		)
-		(property "Description_1" ""
-			(at 43.18 129.54 0)
-			(effects
-				(font
-					(size 1.27 1.27)
-				)
-				(hide yes)
-			)
-		)
-		(property "MANUFACTURER" ""
-			(at 43.18 129.54 0)
-			(effects
-				(font
-					(size 1.27 1.27)
-				)
-				(hide yes)
-			)
-		)
-		(property "MAXIMUM_PACKAGE_HEIGHT" ""
-			(at 43.18 129.54 0)
-			(effects
-				(font
-					(size 1.27 1.27)
-				)
-				(hide yes)
-			)
-		)
-		(property "MF" ""
-			(at 43.18 129.54 0)
-			(effects
-				(font
-					(size 1.27 1.27)
-				)
-				(hide yes)
-			)
-		)
-		(property "MP" ""
-			(at 43.18 129.54 0)
-			(effects
-				(font
-					(size 1.27 1.27)
-				)
-				(hide yes)
-			)
-		)
-		(property "PARTREV" ""
-			(at 43.18 129.54 0)
-			(effects
-				(font
-					(size 1.27 1.27)
-				)
-				(hide yes)
-			)
-		)
-		(property "Package" ""
-			(at 43.18 129.54 0)
-			(effects
-				(font
-					(size 1.27 1.27)
-				)
-				(hide yes)
-			)
-		)
-		(property "Price" ""
-			(at 43.18 129.54 0)
-			(effects
-				(font
-					(size 1.27 1.27)
-				)
-				(hide yes)
-			)
-		)
-		(property "STANDARD" ""
-			(at 43.18 129.54 0)
-			(effects
-				(font
-					(size 1.27 1.27)
-				)
-				(hide yes)
-			)
-		)
-		(property "SnapEDA_Link" ""
-			(at 43.18 129.54 0)
-			(effects
-				(font
-					(size 1.27 1.27)
-				)
-				(hide yes)
-			)
-		)
-		(pin "1"
-		)
-		(instances
-			(project "ponictron"
-				(path "/10078caa-7fd0-475a-83d7-2ff1e936c6b6"
-					(reference "TP1")
-					(unit 1)
-				)

Commit message: Update PCB design to use digipot instead of dac & op-amp
Parts:
- removed C1: 0.1uF, Capacitor_SMD:C_0603_1608Metric, symbol Device:C
- removed C2: 10uF, Capacitor_SMD:C_0603_1608Metric, symbol Device:C
- removed Q1: BSS138, Package_TO_SOT_SMD:SOT-23, symbol Transistor_FET:BSS138
- removed R2: 10kΩ, Resistor_SMD:R_0603_1608Metric_Pad0.98x0.95mm_HandSolder, symbol Device:R
- removed R3: 32kΩ, Resistor_SMD:R_0603_1608Metric_Pad0.98x0.95mm_HandSolder, symbol Device:R
- removed R4: 1kΩ, Resistor_SMD:R_0603_1608Metric_Pad0.98x0.95mm_HandSolder, symbol Device:R
- removed R6: 83Ω, Resistor_SMD:R_0603_1608Metric_Pad0.98x0.95mm_HandSolder, symbol Device:R
- removed U2: MCP4725A1T-E/CH, MCP4725A1T_E_CH:SOT-23-6_MC_MCH, symbol MCP4725A1T_E_CH:MCP4725A1T-E_CH
- removed U3: MCP6001-OT, Package_TO_SOT_SMD:SOT-23-5, symbol Amplifier_Operational:MCP6001-OT
- added U2: DS3502U+T&R, footprints:DS3502U_T_R-L, symbol DS3502U_T_R:DS3502U+T&R
- J11, J5: footprint CONN_SD-47053-001_H10p00_MOL -> 0470531000:CONN_SD-47053-001_H10p00_MOL
- L1: footprint IND_BOURNS_SRR6028 -> SRR6028-3R9Y:IND_BOURNS_SRR6028
- S1, S2: footprint PTS647SM38SMTR2LFS -> SamacSys_Parts:PTS647SM38SMTR2LFS
- U3: renamed from U4; footprint AP63203WU-7_DIO -> AP63203WU-7:AP63203WU-7_DIO-L
- renumbered C4 to C1, C12 to C10, C13 to C11, C14 to C12, C15 to C13, C16 to C14, C17 to C15, C18 to C16, C3 to C2, C5 to C3, C6 to C4, C7 to C5, C8 to C6, C9 to C7, C10 to C8, C11 to C9, Q2 to Q1, R14 to R10, R5 to R2, R7 to R3, R8 to R4, R9 to R5, R10 to R6, R11 to R7, R12 to R8, R13 to R9, TP2 to TP1, TP3 to TP2, TP4 to TP3, U5 to U4, U6 to U5
Connections:
- net +3.3V: now also U2.3 (VCC)
- net GND: now also U2.2 (GND); no longer J1.5
- net SCL: now also U2.10 (SCL)
- net SDA: now also U2.1 (SDA)
- net at J1.6: now also U2.6 (RH)
- new net: J1.5, U2.7 (RW)
Other:
- note removed: "1.2 mA is max current draw of LED sink 0 V -> MOSFET closed -> 0 A -> max brightness 0.1 V / 1.2 mA = 83 Ω 0.1 V -> max current draw -> minimum brightness"
- note removed: "The 83 Ω resistor is what causes the MOSFET to target 0.1 V, given the 1.2 mA. Which in turn drives the 1.2 mA current, Which in turn causes the 10 V drop at the LED driver. You want to target as low of a voltage as possible (0.1 V) so that the required sensing resistance is as low as possible because the 83 Ω gets added to the 8300 Ω 10 V / 8383 Ω = 1.19 mA, so you get as close as possible to ma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"
- note removed: "linear op-amp sink"
- note removed: "voltage divider, 3.3V -> 0.1V"
- moved on the sheet: C1, C2, J1
