File: hw/ponictron.kicad_pcb (KiCad board)
At the start: 2 copper layers, 121 x 73 mm, 75 parts, among them IC1 SHT40-BD1B-R2, IC2 MAX31328NELB+, IC3 PEC11S-929K-S0015, J1 RJCSE538001, J10 B3B-PH-SM4-TB_LF__SN_, J11 470531000, J12 SM04B-SRSS-TB_LF__SN__P_, J13 FC68148S, J2 Conn_01x10, J3 MSD-11-A, J4 B3B-PH-SM4-TB_LF__SN_, J5 470531000, J6 Conn_01x10, J7 B3B-PH-SM4-TB_LF__SN_, J8 B3B-PH-SM4-TB_LF__SN_, J9 B3B-PH-SM4-TB_LF__SN_, Q1 DMG2305UX-7, U1 RaspberryPi_Pico, U2 LM358M, U3 MCP4725A1T-E/CH, U4 AP63203WU-7, U5 NC7WZ14P6X, U6 DMP4015SSSQ-13

Commit message: Various fixes for schematic issues
Parts:
- removed C7, C8: 0.1uF, Capacitor_SMD:C_0603_1608Metric
- removed H1, H2, H3, H4: MountingHole_Pad, 78614015360:WE-SMSA_78614015360
- removed IC3: PEC11S-929K-S0015, SamacSys_Parts:PEC11S929KS0015
- removed R11, R12, R14, R15: 10kΩ, Resistor_SMD:R_0603_1608Metric_Pad0.98x0.95mm_HandSolder
- removed R18: 1kΩ, Resistor_SMD:R_0603_1608Metric_Pad0.98x0.95mm_HandSolder
- removed TP1: Bootsel, TestPoint:TestPoint_Pad_1.5x1.5mm
- removed U2: LM358M, LM358M:8-SOP_OSI
- added MP1: WA-SMSI_9774XXX151, WA-SMSI_9774100151:WA-SMSI_9774100151, F.Cu at (91.8, 53.4)
- added MP2: WA-SMSI_9774XXX151, WA-SMSI_9774100151:WA-SMSI_9774100151, F.Cu at (152.7, 53.4)
- added MP3: WA-SMSI_9774XXX151, WA-SMSI_9774100151:WA-SMSI_9774100151, F.Cu at (152.7, 89.0)
- added MP4: WA-SMSI_9774XXX151, WA-SMSI_9774100151:WA-SMSI_9774100151, F.Cu at (91.8, 89.0)
- added Q2: BSS138, Package_TO_SOT_SMD:SOT-23, F.Cu at (93.6, 36.5)
- added R20: 1kΩ, Resistor_SMD:R_0603_1608Metric_Pad0.98x0.95mm_HandSolder, F.Cu at (93.3, 28.4)
- added U7: MCP6001-OT, Package_TO_SOT_SMD:SOT-23-5, F.Cu at (93.7, 32.1)
- R2: value 2kΩ -> 83Ω
- R3: value 1kΩ -> 32kΩ
- moved R3 68.9 mm to (93.3, 25.9), turned to 0 degrees
- moved R2 67.8 mm to (93.3, 23.4), turned to 0 degrees
- moved J2 22.9 mm to (152.7, 59.8), turned to 0 degrees
Connections:
- C3 pad 2: +12V -> +3.3V
- C4 pad 2: +12V -> +3.3V
- J1 pad 6: Net-(U2-OUT1) -> Net-(Q2-D)
- J11 pad 4: /FAN -> /FAN2
- J13 pad 1: Net-(J13-Pad1) -> GND
- J13 pad 2: Net-(J13-Pad1) -> GND
- J13 pad 4: GND -> Net-(J13-Pad4)
- J3 pad P1: /msdDAT2 -> Net-(J3-DAT2)
- J3 pad P8: /msdDAT1 -> Net-(J3-DAT1)
- J5 pad 4: /FAN -> /FAN1
- R2 pad 1: Net-(U2-OUT1) -> Net-(Q2-S)
- R2 pad 2: Net-(U2-IN1(-)) -> GND
- R3 pad 1: Net-(U2-IN1(-)) -> Net-(U3-VOUT)
- R3 pad 2: GND -> Net-(U7-+)
- R4 pad 2: /msdDAT1 -> Net-(J3-DAT1)
- R6 pad 2: /msdDAT2 -> Net-(J3-DAT2)
- U1 pad 1: /Enc_B1 -> /FAN2
- U1 pad 19: /msdDAT2 -> unconnected-(U1-GPIO14-Pad19)
- U1 pad 2: /Enc_A1 -> unconnected-(U1-GPIO1-Pad2)
- U1 pad 20: /msdDAT1 -> unconnected-(U1-GPIO15-Pad20)
- U1 pad 29: /FAN -> /FAN1
- U1 pad 4: /Enc_E -> unconnected-(U1-GPIO2-Pad4)
- U3 pad 1: Net-(U2-IN1(+)) -> Net-(U3-VOUT)
- U6 pad 5: Net-(J13-Pad1) -> Net-(J13-Pad4)
- U6 pad 6: Net-(J13-Pad1) -> Net-(J13-Pad4)
- U6 pad 7: Net-(J13-Pad1) -> Net-(J13-Pad4)
- U6 pad 8: Net-(J13-Pad1) -> Net-(J13-Pad4)
Routing:
- net /FAN: track 54.6 -> 0.00 mm, vias 1 -> 0
- net /FAN1: track 0.00 -> 47.6 mm, vias 0 -> 1
- net /Enc_E: track 47.3 -> 0.00 mm
- net /SCK: track 97.6 -> 62.2 mm
- net (no net): track 0.00 -> 30.8 mm, vias 0 -> 2
- net Net-(U1-~{BOOTSEL}): track 23.1 -> 0.00 mm
- net /BlitePWM: track 40.8 -> 19.8 mm
- net Net-(IC3-COM): track 20.8 -> 0.00 mm
- net /msdDAT2: track 18.7 -> 0.00 mm, vias 2 -> 0
- net Net-(J13-Pad1): track 14.4 -> 0.00 mm
- net /MOSI: track 102.0 -> 89.7 mm
- net /msdDAT1: track 12.0 -> 0.00 mm
- net Net-(IC3-CCW): track 9.96 -> 0.00 mm
- net Net-(IC3-CW): track 9.88 -> 0.00 mm
- net Net-(U2-OUT1): track 7.95 -> 0.00 mm
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
Commit message: Finish schematic and board layout changes
Parts:
- removed the R10 at (123.4, 61.8)
- removed the U5 at (100.5, 81.0)
- added C5: 10uF, Capacitor_SMD:C_0603_1608Metric, F.Cu at (123.0, 62.5)
- added C6: 0.1uF, Capacitor_SMD:C_0603_1608Metric, F.Cu at (121.0, 62.5)
- added TP1: GP10, TestPoint:TestPoint_Pad_1.5x1.5mm, F.Cu at (135.0, 84.0)
- added TP2: Bootsel, TestPoint:TestPoint_Pad_1.5x1.5mm, F.Cu at (107.5, 109.0)
- added U6: SN74LVC2G240DCUR, SN74LVC2G240DCUR:SN74LVC2G240DCUR, F.Cu at (152.0, 113.0)
- R10: renamed from R9; value 47kΩ -> 10kΩ
- R5: renamed from R4; value 47kΩ -> 10kΩ
- R7: renamed from R5; value 47kΩ -> 10kΩ
- R8: renamed from R6; value 47kΩ -> 10kΩ
- R9: renamed from R8; value 47kΩ -> 10kΩ
- S1, S2: value TL3301BF260QJ -> PTS647SM70SMTR2LFS; footprint SamacSys_Parts:TL3301BF260QJ -> SamacSys_Parts:PTS647SM38SMTR2LFS
- moved LS1 73.3 mm to (164.5, 110.0)
- moved R14 65.1 mm to (155.5, 110.5)
- moved R3 62.0 mm to (83.0, 87.0), turned to 90 degrees
- moved R6 58.2 mm to (89.5, 81.5), turned to -90 degrees
- moved R4 56.8 mm to (88.0, 85.0)
- moved C17 55.0 mm to (152.5, 109.8), turned to -90 degrees
- moved C15 54.3 mm to (150.5, 109.8), turned to -90 degrees
- moved U3 50.0 mm to (86.0, 81.5), turned to 90 degrees
- moved Q1 47.1 mm to (81.5, 82.0), turned to 180 degrees
- moved S2 30.5 mm to (137.4, 111.5), turned to 90 degrees
- moved S1 23.2 mm to (144.4, 111.5), turned to -90 degrees
- moved R10 2.77 mm to (117.2, 62.5)
- moved R8 2.77 mm to (115.5, 62.5)
- moved R9 2.77 mm to (119.0, 62.5)
- moved C4 2.13 mm to (83.0, 78.0)
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- renumbered C2 to C1, C1 to C2, C4 to C3, C3 to C4, C5 to C7, C6 to C8, H5 to H1, H6 to H2, H7 to H3, H8 to H4, Q2 to Q1, Q1 to Q2, R13 to R11, R16 to R12, R17 to R13, R19 to R14, R7 to R2, R20 to R4, R2 to R6, TP2 to TP3, TP3 to TP4, U3 to U2, U7 to U3, U6 to U5
Connections:
- J6 pad 2: GND -> /GP15
- J6 pad 3: GND -> /GP14
- J6 pad 7: /GP7 -> /GP11
- J6 pad 8: /GP6 -> /GP7
- J6 pad 9: +3.3V -> /GP6
- S1 pad 1: /BUT1 -> unconnected-(S1-Pad1)
- S1 pad 2: unconnected-(S1-Pad2) -> GND
- S1 pad 3: unconnected-(S1-Pad3) -> /BUT1
- S1 pad 4: GND -> unconnected-(S1-Pad4)
- S2 pad 1: /BUT2 -> unconnected-(S2-Pad1)
- S2 pad 2: unconnected-(S2-Pad2) -> GND
- S2 pad 3: unconnected-(S2-Pad3) -> /BUT2
- S2 pad 4: GND -> unconnected-(S2-Pad4)
- U1 pad 1: /FAN2 -> /Buzzer
- U1 pad 14: /BUT2 -> Net-(U1-GPIO10)
- U1 pad 15: /BUT1 -> /GP11
- U1 pad 19: unconnected-(U1-GPIO14-Pad19) -> /GP14
- U1 pad 2: unconnected-(U1-GPIO1-Pad2) -> /BUT2
- U1 pad 20: unconnected-(U1-GPIO15-Pad20) -> /GP15
- U1 pad 27: /Buzzer -> /FAN2
- U1 pad 4: unconnected-(U1-GPIO2-Pad4) -> /BUT1
Routing:
- net /FAN2: track 0.00 -> 56.8 mm, vias 0 -> 1
- net /GP14: track 0.00 -> 55.8 mm, vias 0 -> 1
- net /GP15: track 0.00 -> 54.7 mm
- net /GP11: track 0.00 -> 53.7 mm
- net /SCK: track 62.2 -> 107.7 mm, vias 1 -> 0
- net /BUT1: track 54.2 -> 13.8 mm, vias 2 -> 0
- net /BUT2: track 46.9 -> 9.97 mm, vias 2 -> 0
- net (no net): track 30.8 -> 0.00 mm, vias 2 -> 0
- net +12V: track 80.5 -> 50.1 mm
- net Net-(J13-Pad4): track 0.00 -> 24.3 mm, vias 1 -> 0
- net /MOSI: track 89.7 -> 113.7 mm, vias 0 -> 1
- net GND: track 89.4 -> 110.0 mm, vias 27 -> 29
- net Net-(U1-~{BOOTSEL}): track 0.00 -> 17.4 mm
- net /DispD/C: track 23.3 -> 38.0 mm, vias 0 -> 1
- net +3.3V: track 35.4 -> 23.4 mm, vias 9 -> 4
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Other:
- board text added: "BACK"
- board text added: "GP11"
- board text added: "GP14"
- board text added: "GP15"
- board text added: "SAVE"
- board text added: "ponictron v2 Ben Bokser"
- board text removed: "ponictron v1 Ben Bokser"

Commit message: Update schematic and board layout
Parts:
- removed TP1: GP10, TestPoint:TestPoint_Pad_1.5x1.5mm
Connections:
- U1 pad 14: Net-(U1-GPIO10) -> /onewire
- U1 pad 2: /BUT2 -> /Buzzer_EN
- U1 pad 4: /BUT1 -> /BUT2
- U1 pad 5: /onewire -> /BUT1
- U6 pad 1: unconnected-(U6-1OEN-Pad1) -> /Buzzer_EN
- U6 pad 7: unconnected-(U6-2OEN-Pad7) -> /Buzzer_EN
Routing:
- net /Buzzer_EN: track 0.00 -> 25.8 mm
- net /onewire: track 58.9 -> 70.1 mm
- net GND: track 110.0 -> 115.8 mm, vias 29 -> 31
- net Net-(U1-GPIO10): track 4.66 -> 0.00 mm
- net /BUT2: track 9.97 -> 14.2 mm
- net +3.3V: track 23.4 -> 25.5 mm
- net /MOSI: track 113.7 -> 115.8 mm
- net /BUT1: track 13.8 -> 13.2 mm
- net /ADC2: track 64.0 -> 63.4 mm
