File: hw/ponictron.kicad_pcb (KiCad board)
At the start: 2 copper layers, 121 x 73 mm, 70 parts, among them IC1 SHT40-BD1B-R2, IC2 MAX31328NELB+, J1 RJCSE538001, J10 B3B-PH-SM4-TB_LF__SN_, J11 470531000, J12 SM04B-SRSS-TB_LF__SN__P_, J13 FC68148S, J2 Conn_01x10, J3 MSD-11-A, J4 B3B-PH-SM4-TB_LF__SN_, J5 470531000, J6 Conn_01x10, J7 B3B-PH-SM4-TB_LF__SN_, J8 B3B-PH-SM4-TB_LF__SN_, J9 B3B-PH-SM4-TB_LF__SN_, Q1 BSS138, Q2 DMG2305UX-7, U1 RaspberryPi_Pico, U2 MCP4725A1T-E/CH, U3 MCP6001-OT, U4 AP63203WU-7, U5 DMP4015SSSQ-13, U6 SN74LVC2G240DCUR

Commit message: Massive improvement to button press latency via keypad library, and other speed improvements
Parts:
- moved C18 10.3 mm to (100.5, 111.0), turned to -90 degrees
- moved C16 7.75 mm to (98.9, 111.0), turned to -90 degrees
- moved L1 1.50 mm to (94.0, 112.5)
Routing:
- net Net-(Q2-D): track 30.0 -> 15.8 mm
- net GND: track 115.8 -> 117.7 mm, vias 31 -> 29
- net +12V: track 50.1 -> 50.9 mm

Commit message: Update PCB design to use digipot instead of dac & op-amp
Parts:
- removed the C1 at (86.0, 94.2)
- removed the C2 at (82.8, 94.2)
- removed the Q1 at (81.5, 82.0)
- removed the R2 at (86.2, 87.5)
- removed the R3 at (83.0, 87.0)
- removed the R4 at (88.0, 85.0)
- removed the R6 at (89.5, 81.5)
- removed the U3 at (86.0, 81.5)
- U2: value MCP4725A1T-E/CH -> DS3502U+T&R; footprint MCP4725A1T_E_CH:SOT-23-6_MC_MCH -> footprints:DS3502U_T_R-L
- U3: renamed from U4; footprint AP63203WU-7:AP63203WU-7_DIO -> AP63203WU-7:AP63203WU-7_DIO-L
- moved C2 10.4 mm to (89.2, 84.2)
- moved C1 7.70 mm to (87.5, 84.2)
- moved U2 6.49 mm to (83.1, 85.0), turned to 180 degrees
- moved C12 2.55 mm to (96.5, 117.5)
- renumbered C4 to C1, C12 to C10, C13 to C11, C14 to C12, C15 to C13, C16 to C14, C17 to C15, C18 to C16, C3 to C2, C5 to C3, C6 to C4, C7 to C5, C8 to C6, C9 to C7, C10 to C8, C11 to C9, Q2 to Q1, R14 to R10, R5 to R2, R7 to R3, R8 to R4, R9 to R5, R10 to R6, R11 to R7, R12 to R8, R13 to R9, TP2 to TP1, TP3 to TP2, TP4 to TP3, U5 to U4, U6 to U5
Connections:
- J1 pad 5: GND -> Net-(U2-RW)
- J1 pad 6: Net-(Q1-D) (its old number) -> Net-(U2-RH)
- U2 pad 1: Net-(U2-VOUT) -> /SDA
- U2 pad 4: /SDA -> unconnected-(U2-A1-Pad4)
- U2 pad 5: /SCL -> unconnected-(U2-A0-Pad5)
- U2 pad 6: Net-(U2-A0) -> Net-(U2-RH)
Routing:
- net GND: track 117.7 -> 92.0 mm, vias 29 -> 27
- net /SCL: track 113.6 -> 121.6 mm
- net Net-(Q1-S): track 7.81 -> 0.00 mm
- net Net-(U3-+): track 6.96 -> 0.00 mm
- net /SDA: track 112.8 -> 118.7 mm
- net Net-(Q1-D) (its old number): track 4.72 -> 0.00 mm
- net Net-(U2-RH): track 0.00 -> 4.22 mm
- net Net-(U2-RW): track 0.00 -> 4.02 mm
- net Net-(Q1-G): track 2.74 -> 0.00 mm
- net Net-(U2-VOUT): track 2.58 -> 0.00 mm
- net +3.3V: track 25.5 -> 27.8 mm
- net Net-(U2-A0): track 2.10 -> 0.00 mm
- net Net-(U3-BST): track 2.35 -> 4.19 mm
- net Net-(U3-SW): track 10.4 -> 8.85 mm
